Commit message: orange

File: gripper_v2/gripper_description/urdf/finger_segments.xacro (robot description, xacro)
@@ -47,5 +47,5 @@
         </collision>
         <gazebo reference="${prefix}_segment_link_${number}">
-          <material>Gazebo/White</material>
+          <material>Gazebo/Orange</material>
           <mu1>100</mu1>
           <mu2>100</mu2>

Commit message: tidy up

File: gripper_v2/gripper_description/urdf/finger_segments.xacro (robot description, xacro)
@@ -46,12 +46,12 @@
           </geometry>
         </collision>
-        <gazebo reference="${prefix}_segment_link_${number}">
-          <material>Gazebo/Orange</material>
-          <mu1>100</mu1>
-          <mu2>100</mu2>
-          <kp>100</kp>
-          <kd>1</kd>
-        </gazebo>
       </link>
+      <gazebo reference="${prefix}_segment_link_${number}">
+        <material>Gazebo/Orange</material>
+        <!-- <mu1>100</mu1>
+        <mu2>100</mu2>
+        <kp>100</kp>
+        <kd>1</kd> -->
+      </gazebo>
     </xacro:macro>
     <!-- Macro to add a segment joint -->

Commit message: more additions

File: gripper_v2/gripper_description/urdf/finger_segments.xacro (robot description, xacro)
@@ -3,5 +3,4 @@
   <xacro:macro name="segmented_finger" params="prefix num_segments">
     <!-- User defined variables -->
-    <!-- <xacro:property name="num_segments" value="10"/> -->
     <xacro:property name="finger_length_mm" value="190.0"/>
     <xacro:property name="hook_length_mm" value="35.0"/>
@@ -9,9 +8,12 @@
     <xacro:property name="finger_thickness_mm" value="0.9"/>
     <xacro:property name="hook_angle_d" value="90.0"/>
-    <xacro:property name="bending_stiffness" value="100.0"/>
-    <xacro:property name="torsional_stiffness" value="1000.0"/>
-    <xacro:property name="bending_damping" value="0.1"/>
-    <xacro:property name="torsional_damping" value="0.1"/>
+    <xacro:property name="finger_mass_g" value="75.0"/>
+    <!-- set to zero, as handled in segmented_control.h -->
+    <xacro:property name="bending_damping" value="0.0"/>
+    <xacro:property name="torsional_damping" value="0.0"/>
+    <xacro:property name="total_friction" value="0.0"/>
+    <xacro:property name="total_damping" value="0.0001"/>
     <!-- Automatially calculated variables -->
+    <xacro:property name="finger_length" value="${finger_length_mm * 0.001}"/>
     <xacro:property name="segment_length" value="${(finger_length_mm / num_segments) * 0.001}"/>
     <xacro:property name="segment_width" value="${finger_width_mm * 0.001}"/>
@@ -19,11 +21,34 @@
     <xacro:property name="hook_length" value="${hook_length_mm * 0.001}"/>
     <xacro:property name="hook_angle" value="${(hook_angle_d / 180.0) * 3.1415926535897}"/>
-    <xacro:property name="segment_number" value="0"/>
+    <xacro:property name="joint_friction" value="${total_friction / num_segments}"/>
+    <xacro:property name="joint_damping" value="${total_damping * num_segments}"/>
+    <!-- find inertia of each segment -->
+    <xacro:property name="finger_mass" value="${finger_mass_g * 0.001}"/>
+    <xacro:property name="segment_mass"
+      value="${(finger_mass * segment_length) / (finger_length + hook_length)}"/>
+    <!-- x axis along finger length, no axis displacement-->
+    <xacro:property name="segment_ixx"
+      value="${(1.0/12.0) * segment_mass * (segment_thickness ** 2 + segment_width ** 2)}"/>
+    <!-- y axis is joint axis, has axis displacment from centre of mass -->
+    <xacro:property name="segment_iyy"
+      value="${(1.0/12.0) * segment_mass * (segment_length ** 2 + segment_thickness ** 2)
+              + segment_mass * (segment_length / 2.0) ** 2}"/>
+    <!-- z axis is out of the segment, has axis displacement-->
+    <xacro:property name="segment_izz"
+      value="${(1.0/12.0) * segment_mass * (segment_length ** 2 + segment_width ** 2)
+              + segment_mass * (segment_length / 2.0) ** 2}"/>
+    <xacro:property name="stability_factor" value="1"/>
     <!-- Simplistic inertia macro for Gazebo -->
-    <xacro:macro name="segment_inertial" params="mass">
+    <xacro:macro name="segment_inertial" params="mass num">
       <inertial>
-        <mass value="${mass}"/>
-        <inertia ixx="1e-3" iyy="1e-3" izz="1e-3"
+        <mass value="${segment_mass}"/>
+        <inertia ixx="${segment_ixx * stability_factor}"
+                 iyy="${segment_iyy * stability_factor}"
+                 izz="${segment_izz * stability_factor}"
                 ixy="0.00" iyz="0.00" ixz="0.00" />
+        <!-- <inertia ixx="${1e-6 * stability_factor}"
+                 iyy="${1e-6 * stability_factor}"
+                 izz="${1e-6 * stability_factor}"
+                ixy="0.00" iyz="0.00" ixz="0.00" /> -->
       </inertial>
     </xacro:macro>
@@ -31,5 +56,5 @@
     <xacro:macro name="add_segment_link" params="number">
       <link name="${prefix}_segment_link_${number}">
-        <xacro:segment_inertial mass="${(75 * 0.001) / num_segments}"/>
+        <xacro:segment_inertial mass="${(75 * 0.001) / num_segments}" num="${number}"/>
         <visual>
           <origin xyz="${segment_length / 2} 0 0"
@@ -49,7 +74,7 @@
       <gazebo reference="${prefix}_segment_link_${number}">
         <material>Gazebo/Orange</material>
-        <!-- <mu1>100</mu1>
-        <mu2>100</mu2>
-        <kp>100</kp>
+        <mu1>0.1</mu1>
+        <mu2>0.1</mu2>
+        <!-- <kp>100</kp>
         <kd>1</kd> -->
       </gazebo>
@@ -67,27 +92,26 @@
                upper="1.0"
                velocity="1.0"/>
-        <dynamics damping="${bending_damping}"/>
+        <dynamics damping="${joint_damping}" friction="${joint_friction}"/>
+      </joint>
+      <!-- Tags for gazebo, see: http://gazebosim.org/tutorials?tut=ros_urdf -->
+      <xacro:macro name="add_gazebo">
         <gazebo reference="${prefix}_segment_joint_${number - 1}">
-          <spring_reference>0.0</spring_reference>
-          <!-- note series springs have reduced stiffness 10+10+10 = 10/3 -->
-          <spring_stiffness>1000000.0</spring_stiffness>
+          <provideFeedback>1</provideFeedback>
+          <springStiffness>0.75</springStiffness>
+          <springReference>0.0</springReference>
           <implicitSpringDamper>1</implicitSpringDamper>
-          <!-- <stopCfm>0.1</stopCfm>
-          <stopErp>0.1</stopErp>
-          <dampingFactor>0.1</dampingFactor> -->
         </gazebo>
-      </joint>
+      </xacro:macro>
+      <xacro:add_gazebo/>
       <transmission name="${prefix}_segment_tran_${number - 1}">
-          <type>transmission_interface/SimpleTransmission</type>
-          <joint name="${prefix}_segment_joint_${number - 1}">
-                <hardwareInterface>hardware_interface/EffortJointInterface</hardwareInterface>
-          </joint>
-          <actuator name="${prefix}_segment_motor_${number - 1}">
-                <hardwareInterface>hardware_interface/EffortJointInterface</hardwareInterface>
-              <!-- <hardwareInterface>hardware_interface/EffortJointInterface</hardwareInterface> -->
-              <!-- <hardwareInterface>hardware_interface/PositionJointInterface</hardwareInterface> -->
-              <mechanicalReduction>1</mechanicalReduction>
-          </actuator>
-        </transmission>
+        <type>transmission_interface/SimpleTransmission</type>
+        <joint name="${prefix}_segment_joint_${number - 1}">
+          <hardwareInterface>hardware_interface/EffortJointInterface</hardwareInterface>
+        </joint>
+        <actuator name="${prefix}_segment_motor_${number - 1}">
+          <hardwareInterface>hardware_interface/EffortJointInterface</hardwareInterface>
+        <mechanicalReduction>1</mechanicalReduction>
+        </actuator>
+      </transmission>
     </xacro:macro>
     <!-- Create the base link -->
@@ -108,5 +132,5 @@
     <!-- Add the finger hook link -->
     <link name="${prefix}_finger_hook_link">
-      <xacro:segment_inertial mass="${(75 * 0.001) / num_segments}"/>
+      <xacro:segment_inertial mass="${(75 * 0.001) / num_segments}" num="${num_segments}"/>
       <visual>
         <origin xyz="${hook_length / 2} 0 0"
@@ -124,4 +148,11 @@
       </collision>
     </link>
+    <gazebo reference="${prefix}_finger_hook_link">
+      <material>Gazebo/Orange</material>
+      <!-- <mu1>100</mu1>
+      <mu2>100</mu2>
+      <kp>100</kp>
+      <kd>1</kd> -->
+    </gazebo>
     <!-- Connect the finger hook via a fixed joint -->
     <joint name="${prefix}_finger_hook_joint" type="fixed">
@@ -131,8 +162,4 @@
               rpy="0 ${-hook_angle} 0"/>
     </joint>
-    <!-- disable collisions between link and hook -->
-    <disable_collisions link1="${prefix}_segment_link_${num_segments}"
-                        link2="${prefix}_finger_hook_link"
-                        reason="Adjacent"/>
   </xacro:macro>
   <!-- macro to create groups -->
@@ -189,3 +216,9 @@
     <xacro:loop_chain i="${imax}"/>
   </xacro:macro>
+  <!-- macro to include gazebo plugins -->
+  <xacro:macro name="gazebo_plugin">
+    <gazebo>
+      <plugin name="finger_controller_plugin" filename="libfinger_controller_plugin.so"/>
+    </gazebo>
+  </xacro:macro>
 </robot>

File: gripper_v2/gripper_description/urdf/gripper.urdf.xacro (robot description, xacro)
@@ -22,5 +22,5 @@
     <xacro:property name="filename" value="$(find gripper_description)/config/gripper.yaml"/>
     <xacro:property name="dictionary" value="${load_yaml(filename)}"/>
-    <xacro:property name="is_segmented" value="${dictionary['is_segmented']}"/>
+    <xacro:property name="is_segmented" value="${dictionary['gripper_config']['is_segmented']}"/>
     <!-- Define arbritray joint damping for Gazebo -->
     <xacro:property name="joint_damping" value="1.0"/>
@@ -29,11 +29,60 @@
       <inertial>
         <mass value="${mass}"/>
-        <inertia ixx="1e-3" iyy="1e-3" izz="1e-3"
+        <inertia ixx="1e-4" iyy="1e-4" izz="1e-4"
                 ixy="0.00" iyz="0.00" ixz="0.00" />
       </inertial>
     </xacro:macro>
+    <!-- inertias from solidworks -->
+    <xacro:macro name="set_inertia" params="key">
+      <!-- Base-->
+      <xacro:if value="${key == 1}">
+        <inertial>
+          <mass value="1.5"/>
+          <origin xyz="0 0 ${25*0.001}" rpy="${pi} 0 0"/>
+          <inertia ixx="9.95e-3" iyy="10.08e-3" izz="5.13e-3"
+                   ixy="2.73e-6" ixz="-14.32e-6" iyz="121.38e-6"/>
+        </inertial>
+      </xacro:if>
+      <!-- finger intermidiate -->
+      <xacro:if value="${key == 2}">
+        <inertial>
+          <mass value="0.1"/>
+          <origin xyz="0 0 0" rpy="0 0 0"/>
+          <inertia ixx="55.59e-6" iyy="146.36e-6" izz="154.18e-6"
+                   ixy="-47.23e-6" ixz="1.16e-6" iyz="1.00e-6"/>
+        </inertial>
+      </xacro:if>
+      <!-- finger platform no finger (CURRENTLY COPY OF ABOVE) -->
+      <xacro:if value="${key == 3}">
+        <inertial>
+          <mass value="0.1"/>
+          <origin xyz="0 0 0" rpy="0 0 0"/>
+          <inertia ixx="55.59e-6" iyy="146.36e-6" izz="154.18e-6"
+                   ixy="-47.23e-6" ixz="1.16e-6" iyz="1.00e-6"/>
+        </inertial>
+      </xacro:if>
+      <!-- finger platform with finger -->
+      <xacro:if value="${key == 4}">
+        <inertial>
+          <mass value="0.2"/>
+          <origin xyz="0 0 0" rpy="0 0 0"/>
+          <inertia ixx="283.44e-6" iyy="1.38e-3" izz="1.60e-3"
+                   ixy="-567.23e-6" ixz="-6.59e-6" iyz="2.40e-6"/>
+        </inertial>
+      </xacro:if>
+      <!-- palm (CURRENTLY GUESSED)-->
+      <xacro:if value="${key == 5}">
+        <inertial>
+          <mass value="0.05"/>
+          <origin xyz="0 0 0" rpy="0 0 0"/>
+          <inertia ixx="10.0e-6" iyy="10.0e-6" izz="10.0e-6"
+                   ixy="0.0" ixz="0.0" iyz="0.0"/>
+        </inertial>
+      </xacro:if>
+    </xacro:macro>
     <!-- BASE LINK -->
     <link name="gripper_base_link">
-      <xacro:default_inertial mass="1.0"/>
+      <!-- <xacro:default_inertial mass="1.0"/> -->
+      <xacro:set_inertia key="1"/>
       <visual>
         <geometry>
@@ -63,5 +112,6 @@
       <!-- Intermediate link for prismatic joint -->
       <link name="finger_${number}_intermediate">
-        <xacro:default_inertial mass="0.03"/>
+        <!-- <xacro:default_inertial mass="0.03"/> -->
+        <xacro:set_inertia key="2"/>
         <visual>
           <geometry>
@@ -77,7 +127,8 @@
       <!-- Main finger link -->
       <link name="finger_${number}">
-        <xacro:default_inertial mass="0.3"/>
         <!-- If we are using rigid fingers -->
         <xacro:if value="${not is_segmented}">
+          <!-- <xacro:default_inertial mass="0.3"/> -->
+          <xacro:set_inertia key="4"/>
           <visual>
             <geometry>
@@ -93,9 +144,16 @@
         <!-- If we are using segmented fingers -->
         <xacro:if value="${is_segmented}">
+          <!-- <xacro:default_inertial mass="0.3"/> -->
+          <xacro:set_inertia key="3"/>
           <visual>
             <geometry>
-              <mesh filename="package://gripper_description/meshes/finger platform visual.STL"/>
+              <mesh filename="package://gripper_description/meshes/platform only visual.STL"/>
             </geometry>
           </visual>
+          <collision>
+            <geometry>
+              <mesh filename="package://gripper_description/meshes/platform only collision.STL"/>
+            </geometry>
+          </collision>
         </xacro:if>
       </link>
@@ -131,5 +189,6 @@
     <!-- PALM -->
     <link name="palm">
-      <xacro:default_inertial mass="0.05" />
+      <!-- <xacro:default_inertial mass="0.05" /> -->
+      <xacro:set_inertia key="5"/>
       <visual>
         <origin xyz="0 0 0" rpy="0 0 0"/>

File: gripper_v2/gripper_description/urdf/panda_and_eff.xacro (robot description, xacro)
@@ -4,6 +4,6 @@
   <xacro:property name="filename" value="$(find gripper_description)/config/gripper.yaml"/>
   <xacro:property name="dictionary" value="${load_yaml(filename)}"/>
-  <xacro:property name="is_segmented" value="${dictionary['is_segmented']}"/>
-  <xacro:property name="num_segments" value="${dictionary['num_segments']}"/>
+  <xacro:property name="is_segmented" value="${dictionary['gripper_config']['is_segmented']}"/>
+  <xacro:property name="num_segments" value="${dictionary['gripper_config']['num_segments']}"/>
   <!-- include macros for the panda arm and end effector -->
   <xacro:include filename="$(find gripper_description)/urdf/panda_arm_macroed.xacro"/>
@@ -46,4 +46,5 @@
     <xacro:segmented_finger prefix="finger_2" num_segments="${segments}"/>
     <xacro:segmented_finger prefix="finger_3" num_segments="${segments}"/>
+    <xacro:gazebo_plugin/>
     <!-- attach them to the gripper -->
     <joint name="to_segmented_finger_1" type="fixed">

File: gripper_v2/gripper_description/urdf/panda_arm_macroed.xacro (robot description, xacro)
@@ -11,6 +11,39 @@
       </joint>
     </xacro:unless> -->
-    <xacro:macro name="arm_link" params="name visual_mesh:='' collision_mesh:='' mass:='0.0'">
-      <link name="${name}">
+    <!-- added a 5.0N friction tag in the joint macro below -->
+    <xacro:property name="joint_damping" value="1.0"/>
+    <xacro:property name="joint_friction" value="0.0"/>
+    <!-- written by luke based off: https://github.com/justagist/franka_panda_description/blob/master/robots/panda_arm.xacro -->
+    <xacro:macro name="retrieve_inertia" params="link_number">
+      <xacro:if value="${link_number == 0}">
+        <inertia ixx="0.3" ixy="0.0" ixz="0.0" iyy="0.3" iyz="0.0" izz="0.3"/>
+      </xacro:if>
+      <xacro:if value="${link_number == 1}">
+        <inertia ixx="7.0337e-01" ixy="-1.3900e-04" ixz="6.7720e-03" iyy="7.0661e-01" iyz="1.9169e-02" izz="9.1170e-03"/>
+      </xacro:if>
+      <xacro:if value="${link_number == 2}">
+        <inertia ixx="7.9620e-03" ixy="-3.9250e-03" ixz="1.0254e-02" iyy="2.8110e-02" iyz="7.0400e-04" izz="2.5995e-02"/>
+      </xacro:if>
+      <xacro:if value="${link_number == 3}">
+        <inertia ixx="3.7242e-02" ixy="-4.7610e-03" ixz="-1.1396e-02" iyy="3.6155e-02" iyz="-1.2805e-02" izz="1.0830e-02"/>
+      </xacro:if>
+      <xacro:if value="${link_number == 4}">
+        <inertia ixx="2.5853e-02" ixy="7.7960e-03" ixz="-1.3320e-03" iyy="1.9552e-02" iyz="8.6410e-03" izz="2.8323e-02"/>
+      </xacro:if>
+      <xacro:if value="${link_number == 5}">
+        <inertia ixx="3.5549e-02" ixy="-2.1170e-03" ixz="-4.0370e-03" iyy="2.9474e-02" iyz="2.2900e-04" izz="8.6270e-03"/>
+      </xacro:if>
+      <xacro:if value="${link_number == 6}">
+        <inertia ixx="1.9640e-03" ixy="1.0900e-04" ixz="-1.1580e-03" iyy="4.3540e-03" iyz="3.4100e-04" izz="5.4330e-03"/>
+      </xacro:if>
+      <xacro:if value="${link_number == 7}">
+        <inertia ixx="1.2516e-02" ixy="-4.2800e-04" ixz="-1.1960e-03" iyy="1.0027e-02" iyz="-7.4100e-04" izz="4.8150e-03"/>
+      </xacro:if>
+      <xacro:if value="${link_number == 8}">
+        <inertia ixx="1e-4" ixy="0.0" ixz="0.0" iyy="1e-4" iyz="0.0" izz="1e-4"/>
+      </xacro:if>
+    </xacro:macro>
+    <xacro:macro name="arm_link" params="number visual_mesh:='' collision_mesh:='' mass:='0.0'">
+      <link name="${arm_id}_link${number}">
         <xacro:unless value="${not visual_mesh}">
           <visual>
@@ -30,5 +63,6 @@
           <origin xyz="0 0 0" rpy="0 0 0" />
           <mass value="${mass}"/>
-          <inertia ixx="0.3" ixy="0.0" ixz="0.0" iyy="0.3" iyz="0.0" izz="0.3" />
+          <xacro:retrieve_inertia link_number="${number}"/>
+          <!-- <inertia ixx="3e-1" ixy="0.0" ixz="0.0" iyy="3e-1" iyz="0.0" izz="3e-1" /> -->
         </inertial>
       </link>
@@ -51,24 +85,24 @@
           <axis xyz="0 0 0"/>
         </xacro:if>
-        <dynamics damping="1.0"/>
+        <dynamics damping="${joint_damping}" friction="${joint_friction}"/>
       </joint>
     </xacro:macro>
-    <xacro:arm_link name="${arm_id}_link0" visual_mesh="package://${mesh_folder}/visual/link0.dae"
+    <xacro:arm_link number="0" visual_mesh="package://${mesh_folder}/visual/link0.dae"
       collision_mesh="package://${mesh_folder}/collision/link0.stl" mass="3.06"/>
-    <xacro:arm_link name="${arm_id}_link1" visual_mesh="package://${mesh_folder}/visual/link1.dae"
+    <xacro:arm_link number="1" visual_mesh="package://${mesh_folder}/visual/link1.dae"
       collision_mesh="package://${mesh_folder}/collision/link1.stl" mass="2.34"/>
-    <xacro:arm_link name="${arm_id}_link2" visual_mesh="package://${mesh_folder}/visual/link2.dae"
+    <xacro:arm_link number="2" visual_mesh="package://${mesh_folder}/visual/link2.dae"
       collision_mesh="package://${mesh_folder}/collision/link2.stl" mass="2.36"/>
-    <xacro:arm_link name="${arm_id}_link3" visual_mesh="package://${mesh_folder}/visual/link3.dae"
+    <xacro:arm_link number="3" visual_mesh="package://${mesh_folder}/visual/link3.dae"
       collision_mesh="package://${mesh_folder}/collision/link3.stl" mass="2.38"/>
-    <xacro:arm_link name="${arm_id}_link4" visual_mesh="package://${mesh_folder}/visual/link4.dae"
+    <xacro:arm_link number="4" visual_mesh="package://${mesh_folder}/visual/link4.dae"
       collision_mesh="package://${mesh_folder}/collision/link4.stl" mass="2.43"/>
-    <xacro:arm_link name="${arm_id}_link5" visual_mesh="package://${mesh_folder}/visual/link5.dae"
+    <xacro:arm_link number="5" visual_mesh="package://${mesh_folder}/visual/link5.dae"
       collision_mesh="package://${mesh_folder}/collision/link5.stl" mass="3.5"/>
-    <xacro:arm_link name="${arm_id}_link6" visual_mesh="package://${mesh_folder}/visual/link6.dae"
+    <xacro:arm_link number="6" visual_mesh="package://${mesh_folder}/visual/link6.dae"
       collision_mesh="package://${mesh_folder}/collision/link6.stl" mass="1.47"/>
-    <xacro:arm_link name="${arm_id}_link7" visual_mesh="package://${mesh_folder}/visual/link7.dae"
+    <xacro:arm_link number="7" visual_mesh="package://${mesh_folder}/visual/link7.dae"
       collision_mesh="package://${mesh_folder}/collision/link7.stl" mass="0.45"/>
-     <xacro:arm_link name="${arm_id}_link8"/>
+     <xacro:arm_link number="8"/>
      <!-- joint6 limit lower = -0.0175 -->
     <xacro:arm_joint name="${arm_id}_joint1" type="revolute" soft_lower_limit="-2.8973" soft_upper_limit="2.8973"

File: gripper_v2/gripper_moveit/config/robot_model.xacro (robot description, xacro)
@@ -8,6 +8,6 @@
     <xacro:property name="filename" value="$(find gripper_description)/config/gripper.yaml"/>
     <xacro:property name="dictionary" value="${load_yaml(filename)}"/>
-    <xacro:property name="is_segmented" value="${dictionary['is_segmented']}"/>
-    <xacro:property name="num_segments" value="${dictionary['num_segments']}"/>
+    <xacro:property name="is_segmented" value="${dictionary['gripper_config']['is_segmented']}"/>
+    <xacro:property name="num_segments" value="${dictionary['gripper_config']['num_segments']}"/>
     <!-- are we using a segmented finger -->
     <xacro:if value="${is_segmented}">
