Commit message: add meshes

File: gripper_v2/gripper_description/urdf/gripper.urdf.xacro (robot description, xacro)
@@ -34,10 +34,10 @@
       <visual>
         <geometry>
-          <mesh filename="package://gripper_test/meshes/main body visual.STL"/>
+          <mesh filename="package://gripper_description/meshes/main body visual.STL"/>
         </geometry>
       </visual>
       <collision>
         <geometry>
-          <mesh filename="package://gripper_test/meshes/main body collision.STL"/>
+          <mesh filename="package://gripper_description/meshes/main body collision.STL"/>
         </geometry>
       </collision>
@@ -62,10 +62,10 @@
         <visual>
           <geometry>
-            <mesh filename="package://gripper_test/meshes/nut visual.STL"/>
+            <mesh filename="package://gripper_description/meshes/nut visual.STL"/>
           </geometry>
         </visual>
         <collision>
           <geometry>
-            <mesh filename="package://gripper_test/meshes/nut collision.STL"/>
+            <mesh filename="package://gripper_description/meshes/nut collision.STL"/>
           </geometry>
         </collision>
@@ -76,10 +76,10 @@
         <visual>
           <geometry>
-            <mesh filename="package://gripper_test/meshes/finger platform visual.STL"/>
+            <mesh filename="package://gripper_description/meshes/finger platform visual.STL"/>
           </geometry>
         </visual>
         <!-- <collision>
           <geometry>
-            <mesh filename="package://gripper_test/meshes/finger platform collision.STL"/>
+            <mesh filename="package://gripper_description/meshes/finger platform collision.STL"/>
           </geometry>
         </collision> -->
@@ -120,10 +120,10 @@
         <origin xyz="0 0 0" rpy="0 0 0"/>
         <geometry>
-          <mesh filename="package://gripper_test/meshes/palm visual.STL" />
+          <mesh filename="package://gripper_description/meshes/palm visual.STL" />
         </geometry>
       </visual>
       <collision>
         <geometry>
-          <mesh filename="package://gripper_test/meshes/palm collision.STL" />
+          <mesh filename="package://gripper_description/meshes/palm collision.STL" />
         </geometry>
       </collision>

File: gripper_v2/gripper_description/urdf/panda_and_eff.xacro (robot description, xacro)
@@ -14,5 +14,5 @@
     <xacro:my_gripper/>
     <!-- <link name="base_link"/> -->
-    <xacro:panda_arm arm_id="panda" mesh_folder="gripper_test/meshes_panda" connected_to="base_link" xyz="0 0 0" rpy="0 0 0"/>
+    <xacro:panda_arm arm_id="panda" mesh_folder="gripper_description/meshes_panda" connected_to="base_link" xyz="0 0 0" rpy="0 0 0"/>
     <!-- attach panda arm to the ground for gazebo -->
     <link name="world"/>

Commit message: more scripting

File: gripper_v2/gripper_description/urdf/gripper.urdf.xacro (robot description, xacro)
@@ -19,4 +19,8 @@
     <xacro:property name="limit_effort_revolute" value="40.0"/>
     <xacro:property name="limit_effort_palm" value="40.0"/>
+    <!-- retrieve info about the gripper -->
+    <xacro:property name="filename" value="$(find gripper_description)/config/gripper.yaml"/>
+    <xacro:property name="dictionary" value="${load_yaml(filename)}"/>
+    <xacro:property name="is_segmented" value="${dictionary['is_segmented']}"/>
     <!-- Define arbritray joint damping for Gazebo -->
     <xacro:property name="joint_damping" value="1.0"/>
@@ -74,14 +78,25 @@
       <link name="finger_${number}">
         <xacro:default_inertial mass="0.3"/>
-        <visual>
-          <geometry>
-            <mesh filename="package://gripper_description/meshes/finger platform visual.STL"/>
-          </geometry>
-        </visual>
-        <!-- <collision>
-          <geometry>
-            <mesh filename="package://gripper_description/meshes/finger platform collision.STL"/>
-          </geometry>
-        </collision> -->
+        <!-- If we are using rigid fingers -->
+        <xacro:if value="${not is_segmented}">
+          <visual>
+            <geometry>
+              <mesh filename="package://gripper_description/meshes/finger platform visual.STL"/>
+            </geometry>
+          </visual>
+          <collision>
+            <geometry>
+              <mesh filename="package://gripper_description/meshes/finger platform collision.STL"/>
+            </geometry>
+          </collision>
+        </xacro:if>
+        <!-- If we are using segmented fingers -->
+        <xacro:if value="${is_segmented}">
+          <visual>
+            <geometry>
+              <mesh filename="package://gripper_description/meshes/finger platform visual.STL"/>
+            </geometry>
+          </visual>
+        </xacro:if>
       </link>
       <!-- Prismatic joint -->

File: gripper_v2/gripper_description/urdf/panda_and_eff.xacro (robot description, xacro)
@@ -1,4 +1,9 @@
 <?xml version="1.0"?>
 <robot name="gripper" xmlns:xacro="http://wiki.ros.org/xacro">
+  <!-- load information from the gripper yaml file -->
+  <xacro:property name="filename" value="$(find gripper_description)/config/gripper.yaml"/>
+  <xacro:property name="dictionary" value="${load_yaml(filename)}"/>
+  <xacro:property name="is_segmented" value="${dictionary['is_segmented']}"/>
+  <xacro:property name="num_segments" value="${dictionary['num_segments']}"/>
   <!-- include macros for the panda arm and end effector -->
   <xacro:include filename="$(find gripper_description)/urdf/panda_arm_macroed.xacro"/>
@@ -35,7 +40,7 @@
   <xacro:panda_with_eff/>
   <!-- TESTING segmented finger -->
-  <xacro:macro name="add_fingers">
+  <xacro:macro name="add_fingers" params="segments">
     <!-- Create the fingers -->
-    <xacro:property name="segments" value="10"/>
+    <!-- <xacro:property name="segments" value="10"/> -->
     <xacro:segmented_finger prefix="finger_1" num_segments="${segments}"/>
     <xacro:segmented_finger prefix="finger_2" num_segments="${segments}"/>
@@ -57,22 +62,7 @@
       <child link="finger_3_segment_link_1"/>
     </joint>
-    <!-- disable collisions -->
-    <!-- <disable_collisions link1="finger_1"
-                        link2="finger_1_segment_link_1"
-                        reason="Adjacent"/>
-    <disable_collisions link1="finger_2"
-                        link2="finger_2_segment_link_1"
-                        reason="Adjacent"/>
-    <disable_collisions link1="finger_3"
-                        link2="finger_3_segment_link_1"
-                        reason="Adjacent"/> -->
-    <!-- create groups -->
-    <!-- <xacro:build_group prefix="finger_1" i="${segments}"/>
-    <xacro:build_group prefix="finger_2" i="${segments}"/>
-    <xacro:build_group prefix="finger_3" i="${segments}"/> -->
-    <!-- <xacro:disable_finger_collisions prefix="finger_1" imax="2"/>
-	<xacro:disable_finger_collisions prefix="finger_2" imax="2"/>
-	<xacro:disable_finger_collisions prefix="finger_3" imax="2"/> -->
   </xacro:macro>
-  <xacro:add_fingers/>
+  <xacro:if value="${is_segmented}">
+    <xacro:add_fingers segments="${num_segments}"/>
+  </xacro:if>
 </robot>

File: gripper_v2/gripper_moveit/config/robot_model.xacro (robot description, xacro)
@@ -5,12 +5,22 @@
 -->
 <robot name="panda" xmlns:xacro="http://ros.org/wiki/xacro">
-	<xacro:include filename="$(find gripper_description)/urdf/finger_segments.xacro"/>
-	<xacro:property name="num_segments" value="10"/>
-	<xacro:build_group prefix="finger_1" i="${num_segments}"/>
-	<xacro:build_group prefix="finger_2" i="${num_segments}"/>
-	<xacro:build_group prefix="finger_3" i="${num_segments}"/>
-	<xacro:disable_finger_collisions prefix="finger_1" imax="${num_segments}"/>
-	<xacro:disable_finger_collisions prefix="finger_2" imax="${num_segments}"/>
-	<xacro:disable_finger_collisions prefix="finger_3" imax="${num_segments}"/>
+    <!-- retrieve info about the gripper -->
+    <xacro:property name="filename" value="$(find gripper_description)/config/gripper.yaml"/>
+    <xacro:property name="dictionary" value="${load_yaml(filename)}"/>
+    <xacro:property name="is_segmented" value="${dictionary['is_segmented']}"/>
+    <xacro:property name="num_segments" value="${dictionary['num_segments']}"/>
+    <!-- are we using a segmented finger -->
+    <xacro:if value="${is_segmented}">
+        <!-- import gripper macros -->
+        <xacro:include filename="$(find gripper_description)/urdf/finger_segments.xacro"/>
+        <!-- create move groups for each finger -->
+        <xacro:build_group prefix="finger_1" i="${num_segments}"/>
+        <xacro:build_group prefix="finger_2" i="${num_segments}"/>
+        <xacro:build_group prefix="finger_3" i="${num_segments}"/>
+        <!-- disable all possible finger self-collisions -->
+        <xacro:disable_finger_collisions prefix="finger_1" imax="${num_segments}"/>
+        <xacro:disable_finger_collisions prefix="finger_2" imax="${num_segments}"/>
+        <xacro:disable_finger_collisions prefix="finger_3" imax="${num_segments}"/>
+    </xacro:if>
     <!--GROUPS: Representation of a set of joints and links. This can be useful for specifying DOF to plan for, defining arms, end effectors, etc-->
     <!--LINKS: When a link is specified, the parent joint of that link (if it exists) is automatically included-->
@@ -161,59 +171,3 @@
     <disable_collisions link1="panda_link5" link2="panda_link7" reason="Never" />
     <disable_collisions link1="panda_link6" link2="panda_link7" reason="Adjacent" />
-    <!-- disable collisions
-    <disable_collisions link1="finger_1"
-                        link2="finger_1_segment_link_1"
-                        reason="Adjacent"/>
-    <disable_collisions link1="finger_2"
-                        link2="finger_2_segment_link_1"
-                        reason="Adjacent"/>
-    <disable_collisions link1="finger_3"
-                        link2="finger_3_segment_link_1"
-                        reason="Adjacent"/>
-    <disable_collisions link1="finger_1_segment_link_1"
-                        link2="finger_1_segment_link_2"
-                        reason="Adjacent"/>
-    <disable_collisions link1="finger_2_segment_link_1"
-                        link2="finger_2_segment_link_2"
-                        reason="Adjacent"/>
-    <disable_collisions link1="finger_3_segment_link_1"
-                        link2="finger_3_segment_link_2"
-                        reason="Adjacent"/>
-    <disable_collisions link1="finger_1"
-                        link2="finger_1_segment_link_2"
-                        reason="Adjacent"/>
-    <disable_collisions link1="finger_2"
-                        link2="finger_2_segment_link_2"
-                        reason="Adjacent"/>
-    <disable_collisions link1="finger_3"
-                        link2="finger_3_segment_link_2"
-                        reason="Adjacent"/>
-    <disable_collisions link1="finger_1_finger_hook_link"
-                        link2="finger_1_segment_link_2"
-                        reason="Adjacent"/>
-    <disable_collisions link1="finger_2_finger_hook_link"
-                        link2="finger_2_segment_link_2"
-                        reason="Adjacent"/>
-    <disable_collisions link1="finger_3_finger_hook_link"
-                        link2="finger_3_segment_link_2"
-                        reason="Adjacent"/>
-    <disable_collisions link1="finger_1_finger_hook_link"
-                        link2="finger_1"
-                        reason="Adjacent"/>
-    <disable_collisions link1="finger_2_finger_hook_link"
-                        link2="finger_2"
-                        reason="Adjacent"/>
-    <disable_collisions link1="finger_3_finger_hook_link"
-                        link2="finger_3"
-                        reason="Adjacent"/>
-    <disable_collisions link1="finger_1_finger_hook_link"
-                        link2="finger_1_segment_link_1"
-                        reason="Adjacent"/>
-    <disable_collisions link1="finger_2_finger_hook_link"
-                        link2="finger_2_segment_link_1"
-                        reason="Adjacent"/>
-    <disable_collisions link1="finger_3_finger_hook_link"
-                        link2="finger_3_segment_link_1"
-                        reason="Adjacent"/>
-                        -->
 </robot>
