Commit message: tidy

File: gripper_v2/gripper_description/urdf/gripper.urdf.xacro (robot description, xacro)
@@ -1,217 +1,12 @@
 <?xml version="1.0"?>
-<robot xmlns:xacro="http://ros.org/wiki/xacro">
-  <xacro:macro name="my_gripper">
-    <!-- Constants for specifying finger start position, no need to change -->
-    <xacro:property name="radius" value="0.0"/>
-    <xacro:property name="angle" value="0.0"/>
-    <!-- Define motion limits of each joint -->
-    <xacro:property name="finger_displacement_min" value="0.053"/>
-    <xacro:property name="finger_displacement_max" value="0.141"/>
-    <xacro:property name="finger_angle_min" value="-0.7"/>
-    <xacro:property name="finger_angle_max" value="0.7"/>
-    <xacro:property name="palm_displacement_min" value="0.0"/>
-    <xacro:property name="palm_displacement_max" value="0.16"/>
-    <!-- Define limits of each joint -->
-    <xacro:property name="finger_displacement_velocity" value="0.015"/>
-    <xacro:property name="finger_angle_velocity" value="0.1"/>
-    <xacro:property name="palm_velocity" value="0.036"/>
-    <xacro:property name="limit_effort_prismatic" value="40.0"/>
-    <xacro:property name="limit_effort_revolute" value="40.0"/>
-    <xacro:property name="limit_effort_palm" value="40.0"/>
-    <!-- retrieve info about the gripper -->
-    <xacro:property name="filename" value="$(find gripper_description)/config/gripper.yaml"/>
-    <xacro:property name="dictionary" value="${load_yaml(filename)}"/>
-    <xacro:property name="is_segmented" value="${dictionary['gripper_config']['is_segmented']}"/>
-    <!-- Define arbritray joint damping for Gazebo -->
-    <xacro:property name="joint_damping" value="1.0"/>
-	  <!-- Simplistic inertia macro for Gazebo -->
-    <xacro:macro name="default_inertial" params="mass">
-      <inertial>
-        <mass value="${mass}"/>
-        <inertia ixx="1e-4" iyy="1e-4" izz="1e-4"
-                ixy="0.00" iyz="0.00" ixz="0.00" />
-      </inertial>
-    </xacro:macro>
-    <!-- inertias from solidworks -->
-    <xacro:macro name="set_inertia" params="key">
-      <!-- Base-->
-      <xacro:if value="${key == 1}">
-        <inertial>
-          <mass value="1.5"/>
-          <origin xyz="0 0 ${25*0.001}" rpy="${pi} 0 0"/>
-          <inertia ixx="9.95e-3" iyy="10.08e-3" izz="5.13e-3"
-                   ixy="2.73e-6" ixz="-14.32e-6" iyz="121.38e-6"/>
-        </inertial>
-      </xacro:if>
-      <!-- finger intermidiate -->
-      <xacro:if value="${key == 2}">
-        <inertial>
-          <mass value="0.1"/>
-          <origin xyz="0 0 0" rpy="0 0 0"/>
-          <inertia ixx="55.59e-6" iyy="146.36e-6" izz="154.18e-6"
-                   ixy="-47.23e-6" ixz="1.16e-6" iyz="1.00e-6"/>
-        </inertial>
-      </xacro:if>
-      <!-- finger platform no finger (CURRENTLY COPY OF ABOVE) -->
-      <xacro:if value="${key == 3}">
-        <inertial>
-          <mass value="0.1"/>
-          <origin xyz="0 0 0" rpy="0 0 0"/>
-          <inertia ixx="55.59e-6" iyy="146.36e-6" izz="154.18e-6"
-                   ixy="-47.23e-6" ixz="1.16e-6" iyz="1.00e-6"/>
-        </inertial>
-      </xacro:if>
-      <!-- finger platform with finger -->
-      <xacro:if value="${key == 4}">
-        <inertial>
-          <mass value="0.2"/>
-          <origin xyz="0 0 0" rpy="0 0 0"/>
-          <inertia ixx="283.44e-6" iyy="1.38e-3" izz="1.60e-3"
-                   ixy="-567.23e-6" ixz="-6.59e-6" iyz="2.40e-6"/>
-        </inertial>
-      </xacro:if>
-      <!-- palm (CURRENTLY GUESSED)-->
-      <xacro:if value="${key == 5}">
-        <inertial>
-          <mass value="0.05"/>
-          <origin xyz="0 0 0" rpy="0 0 0"/>
-          <inertia ixx="10.0e-6" iyy="10.0e-6" izz="10.0e-6"
-                   ixy="0.0" ixz="0.0" iyz="0.0"/>
-        </inertial>
-      </xacro:if>
-    </xacro:macro>
-    <!-- BASE LINK -->
-    <link name="gripper_base_link">
-      <!-- <xacro:default_inertial mass="1.0"/> -->
-      <xacro:set_inertia key="1"/>
-      <visual>
-        <geometry>
-          <mesh filename="package://gripper_description/meshes/main body visual.STL"/>
-        </geometry>
-      </visual>
-      <collision>
-        <geometry>
-          <mesh filename="package://gripper_description/meshes/main body collision.STL"/>
-        </geometry>
-      </collision>
-    </link>
-    <!-- Finger position macros -->
-    <xacro:macro name="finger_intermediate_origin" params="number">
-      <origin xyz="${radius * sin((number-1)*((2*pi)/3))}
-                   ${radius * cos((number-1)*((2*pi)/3))}
-                   0"
-              rpy="${3*pi/2}
-                   ${3*pi/2}
-                   ${(pi/2) - (number-1)*(2*pi/3)}" />
-    </xacro:macro>
-    <xacro:macro name="finger_origin" params="number">
-      <origin xyz="0 0 0" rpy="0 0 ${angle}" />
-    </xacro:macro>
-    <!-- Finger Macro -->
-    <xacro:macro name="finger" params="number">
-      <!-- Intermediate link for prismatic joint -->
-      <link name="finger_${number}_intermediate">
-        <!-- <xacro:default_inertial mass="0.03"/> -->
-        <xacro:set_inertia key="2"/>
-        <visual>
-          <geometry>
-            <mesh filename="package://gripper_description/meshes/nut visual.STL"/>
-          </geometry>
-        </visual>
-        <collision>
-          <geometry>
-            <mesh filename="package://gripper_description/meshes/nut collision.STL"/>
-          </geometry>
-        </collision>
-      </link>
-      <!-- Main finger link -->
-      <link name="finger_${number}">
-        <!-- If we are using rigid fingers -->
-        <xacro:if value="${not is_segmented}">
-          <!-- <xacro:default_inertial mass="0.3"/> -->
-          <xacro:set_inertia key="4"/>
-          <visual>
-            <geometry>
-              <mesh filename="package://gripper_description/meshes/finger platform visual.STL"/>
-            </geometry>
-          </visual>
-          <collision>
-            <geometry>
-              <mesh filename="package://gripper_description/meshes/finger platform collision.STL"/>
-            </geometry>
-          </collision>
-        </xacro:if>
-        <!-- If we are using segmented fingers -->
-        <xacro:if value="${is_segmented}">
-          <!-- <xacro:default_inertial mass="0.3"/> -->
-          <xacro:set_inertia key="3"/>
-          <visual>
-            <geometry>
-              <mesh filename="package://gripper_description/meshes/platform only visual.STL"/>
-            </geometry>
-          </visual>
-          <collision>
-            <geometry>
-              <mesh filename="package://gripper_description/meshes/platform only collision.STL"/>
-            </geometry>
-          </collision>
-        </xacro:if>
-      </link>
-      <!-- Prismatic joint -->
-      <joint name="finger_${number}_prismatic_joint" type="prismatic">
-        <axis xyz="0 1 0" rpy="0 0 0"/>
-        <parent link="gripper_base_link"/>
-        <child link="finger_${number}_intermediate"/>
-        <xacro:finger_intermediate_origin number="${number}"/>
-        <limit effort="${limit_effort_prismatic}"
-        			 lower="${finger_displacement_min}"
-        			 upper="${finger_displacement_max}"
-        			 velocity="${finger_displacement_velocity}"/>
-        <dynamics damping="${joint_damping}"/>
-      </joint>
-      <!-- Revolute joint -->
-      <joint name="finger_${number}_revolute_joint" type="revolute">
-        <axis xyz="0 0 1" rpy="0 0 0"/>
-        <parent link="finger_${number}_intermediate"/>
-        <child link="finger_${number}"/>
-        <xacro:finger_origin number="${number}"/>
-        <limit effort="${limit_effort_revolute}"
-        			 lower="${finger_angle_min}"
-        			 upper="${finger_angle_max}"
-        			 velocity="${finger_angle_velocity}"/>
-        <dynamics damping="${joint_damping}"/>
-      </joint>
-    </xacro:macro>
-    <!-- FINGERS -->
-    <xacro:finger number="1"/>
-    <xacro:finger number="2"/>
-    <xacro:finger number="3"/>
-    <!-- PALM -->
-    <link name="palm">
-      <!-- <xacro:default_inertial mass="0.05" /> -->
-      <xacro:set_inertia key="5"/>
-      <visual>
-        <origin xyz="0 0 0" rpy="0 0 0"/>
-        <geometry>
-          <mesh filename="package://gripper_description/meshes/palm visual.STL" />
-        </geometry>
-      </visual>
-      <collision>
-        <geometry>
-          <mesh filename="package://gripper_description/meshes/palm collision.STL" />
-        </geometry>
-      </collision>
-    </link>
-    <joint name="palm_prismatic_joint" type="prismatic">
-      <axis xyz="1 0 0" rpy="0 0 0" />
-      <parent link="gripper_base_link"/>
-      <child link="palm"/>
-      <origin xyz="0 0 0" rpy="0 ${-pi/2} 0"/>
-      <limit effort="${limit_effort_palm}"
-      			 lower="${palm_displacement_min}"
-      			 upper="${palm_displacement_max}"
-      			 velocity="${palm_velocity}"/>
-      <dynamics damping="${joint_damping}"/>
-    </joint>
-  </xacro:macro>
+<robot name="gripper" xmlns:xacro="http://wiki.ros.org/xacro">
+	<xacro:include filename="$(find gripper_description)/xacro/gripper.xacro"/>
+	<xacro:add_gripper/>
+	<!-- attach gripper to the ground for gazebo -->
+	<link name="world"/>
+	<joint name="world_to_base" type="fixed">
+		<origin xyz="0 0 1" rpy="${pi} 0 0"/>
+		<parent link="world"/>
+		<child link="gripper_base_link"/>
+	</joint>
 </robot>

File: gripper_v2/gripper_description/xacro/semantic/add_gripper_config.xacro (robot description, xacro)
@@ -14,5 +14,5 @@
 		  <xacro:if value="${is_segmented}">
 		      <!-- import gripper macros -->
-		      <xacro:include filename="$(find gripper_description)/urdf/finger_segments.xacro"/>
+		      <xacro:include filename="$(find gripper_description)/xacro/gripper.segmented_fingers.xacro"/>
 		      <!-- create move groups for each finger -->
 		      <xacro:build_group prefix="finger_1" i="${num_segments}"/>

File: gripper_v2/gripper_description/xacro/semantic/gripper.semantic.xacro (robot description, xacro)
@@ -6,5 +6,5 @@
 <robot name="gripper" xmlns:xacro="http://ros.org/wiki/xacro">
 		<!-- load the gripper xacro -->
-		<xacro:include filename="$(find gripper_description)/moveit_xacros/add_gripper_config.xacro"/>
+		<xacro:include filename="$(find gripper_description)/xacro/semantic/add_gripper_config.xacro"/>
 		<!-- run the macros -->
 		<xacro:add_gripper_config/>

File: gripper_v2/gripper_description/xacro/semantic/panda.semantic.xacro (robot description, xacro)
@@ -6,5 +6,5 @@
 <robot name="panda" xmlns:xacro="http://ros.org/wiki/xacro">
 		<!-- load the panda xacro -->
-		<xacro:include filename="$(find gripper_description)/moveit_xacros/add_panda_config.xacro"/>
+		<xacro:include filename="$(find gripper_description)/xacro/semantic/add_panda_config.xacro"/>
 		<!-- run the macros -->
 		<xacro:add_panda_config/>

File: gripper_v2/gripper_description/xacro/semantic/panda_and_gripper.semantic.xacro (robot description, xacro)
@@ -6,6 +6,6 @@
 <robot name="panda_and_gripper" xmlns:xacro="http://ros.org/wiki/xacro">
 		<!-- load the gripper and panda xacros -->
-		<xacro:include filename="$(find gripper_description)/moveit_xacros/add_gripper_config.xacro"/>
-		<xacro:include filename="$(find gripper_description)/moveit_xacros/add_panda_config.xacro"/>
+		<xacro:include filename="$(find gripper_description)/xacro/semantic/add_gripper_config.xacro"/>
+		<xacro:include filename="$(find gripper_description)/xacro/semantic/add_panda_config.xacro"/>
 		<!-- run the macros -->
 		<xacro:add_gripper_config/>
