Commit message: more

File: gripper_v2/gripper_description/urdf/panda.urdf (robot description, URDF)
Before this commit: robot panda, 10 links, 9 joints
Links:
- link panda_link0: geometry collision mesh filename=package://gripper_description/meshes_panda/panda collision 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; visual mesh filename=package://gripper_description/meshes_panda/panda visual lin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
- link panda_link1: geometry collision mesh filename=package://gripper_description/meshes_panda/panda collision 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; visual mesh filename=package://gripper_description/meshes_panda/panda visual lin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
- link panda_link2: geometry collision mesh filename=package://gripper_description/meshes_panda/panda collision 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; visual mesh filename=package://gripper_description/meshes_panda/panda visual lin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
- link panda_link3: geometry collision mesh filename=package://gripper_description/meshes_panda/panda collision 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; visual mesh filename=package://gripper_description/meshes_panda/panda visual lin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
- link panda_link4: geometry collision mesh filename=package://gripper_description/meshes_panda/panda collision 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; visual mesh filename=package://gripper_description/meshes_panda/panda visual lin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
- link panda_link5: geometry collision mesh filename=package://gripper_description/meshes_panda/panda collision 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; visual mesh filename=package://gripper_description/meshes_panda/panda visual lin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
- link panda_link6: geometry collision mesh filename=package://gripper_description/meshes_panda/panda collision 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; visual mesh filename=package://gripper_description/meshes_panda/panda visual lin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
- link panda_link7: geometry collision mesh filename=package://gripper_description/meshes_panda/panda collision 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; visual mesh filename=package://gripper_description/meshes_panda/panda visual lin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

File: gripper_v2/gripper_description/urdf/panda_and_gripper.urdf (robot description, URDF)
Before this commit: robot panda_and_gripper, 51 links, 50 joints
Links:
- link panda_link0: geometry collision mesh filename=package://gripper_description/meshes_panda/panda collision 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; visual mesh filename=package://gripper_description/meshes_panda/panda visual lin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
- link panda_link1: geometry collision mesh filename=package://gripper_description/meshes_panda/panda collision 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; visual mesh filename=package://gripper_description/meshes_panda/panda visual lin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
- link panda_link2: geometry collision mesh filename=package://gripper_description/meshes_panda/panda collision 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; visual mesh filename=package://gripper_description/meshes_panda/panda visual lin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
- link panda_link3: geometry collision mesh filename=package://gripper_description/meshes_panda/panda collision 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; visual mesh filename=package://gripper_description/meshes_panda/panda visual lin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
- link panda_link4: geometry collision mesh filename=package://gripper_description/meshes_panda/panda collision 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; visual mesh filename=package://gripper_description/meshes_panda/panda visual lin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
- link panda_link5: geometry collision mesh filename=package://gripper_description/meshes_panda/panda collision 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; visual mesh filename=package://gripper_description/meshes_panda/panda visual lin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
- link panda_link6: geometry collision mesh filename=package://gripper_description/meshes_panda/panda collision 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; visual mesh filename=package://gripper_description/meshes_panda/panda visual lin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
- link panda_link7: geometry collision mesh filename=package://gripper_description/meshes_panda/panda collision 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; visual mesh filename=package://gripper_description/meshes_panda/panda visual lin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
Joints:
- removed joint panda_to_eef_base_link
- added joint panda_to_eef_base_joint: type fixed, parent panda_link7, child gripper_base_link, origin xyz=0 0 0.25 rpy=0 0 -0.785398163397

File: gripper_v2/gripper_description/urdf/panda_and_gripper.urdf.xacro (robot description, xacro)
@@ -16,8 +16,11 @@
 	<!-- connect the gripper to the panda -->
 	<!-- TODO verify these values, change panda_link7 to 8 -->
-  <joint name="panda_to_eef_base_link" type="fixed">
+  <joint name="panda_to_eef_base_joint" type="fixed">
     <origin xyz="0 0 0.25" rpy="0 0 ${-pi/4}" />
     <parent link="panda_link7"/>
     <child link="gripper_base_link"/>
   </joint>
+	<gazebo>
+		<plugin name="reset_joints_plugin" filename="libreset_joints_plugin.so"/>
+	</gazebo>
 </robot>

File: gripper_v2/gripper_description/xacro/gripper.main.xacro (robot description, xacro)
@@ -2,8 +2,11 @@
 <robot xmlns:xacro="http://ros.org/wiki/xacro">
   <xacro:macro name="gripper" params="is_segmented">
-    <!-- Constants for specifying finger start position, no need to change -->
-    <xacro:property name="radius" value="0.0"/>
-    <xacro:property name="angle" value="0.0"/>
-    <!-- Define motion limits of each joint -->
+  	<!-- retrieve info about the gripper
+    <xacro:property name="filename" value="$(find gripper_description)/config/gripper.yaml"/>
+    <xacro:property name="dictionary" value="${xacro.load_yaml(filename)}"/>
+    <xacro:property name="is_segmented" value="${dictionary['gripper_config']['is_segmented']}"/>
+    -->
+  	<!-- PARAMETERS TO BE SET BY HAND -->
+    <!-- Define motion limits of each joint, these all in SI units -->
     <xacro:property name="finger_displacement_min" value="0.053"/>
     <xacro:property name="finger_displacement_max" value="0.141"/>
@@ -12,5 +15,5 @@
     <xacro:property name="palm_displacement_min" value="0.0"/>
     <xacro:property name="palm_displacement_max" value="0.16"/>
-    <!-- Define limits of each joint -->
+    <!-- Define limits of each joint, these all in SI units -->
     <xacro:property name="finger_displacement_velocity" value="0.015"/>
     <xacro:property name="finger_angle_velocity" value="0.1"/>
@@ -19,12 +22,59 @@
     <xacro:property name="limit_effort_revolute" value="40.0"/>
     <xacro:property name="limit_effort_palm" value="40.0"/>
-    <!-- retrieve info about the gripper
-    <xacro:property name="filename" value="$(find gripper_description)/config/gripper.yaml"/>
-    <xacro:property name="dictionary" value="${load_yaml(filename)}"/>
-    <xacro:property name="is_segmented" value="${dictionary['gripper_config']['is_segmented']}"/>
-    -->
-    <!-- Define arbritray joint damping for Gazebo -->
+		<!-- Define arbritray joint damping for Gazebo -->
     <xacro:property name="joint_damping" value="1.0"/>
-	  <!-- Simplistic inertia macro for Gazebo -->
+    <!-- inertias from solidworks -->
+    <xacro:macro name="set_inertia" params="key">
+      <!-- Base-->
+      <xacro:if value="${key == 1}">
+        <inertial>
+          <mass value="1.5"/>
+          <origin xyz="0 0 ${25*0.001}" rpy="${pi} 0 0"/>
+          <inertia ixx="9.95e-3" iyy="10.08e-3" izz="5.13e-3"
+                   ixy="2.73e-6" ixz="-14.32e-6" iyz="121.38e-6"/>
+        </inertial>
+      </xacro:if>
+      <!-- finger intermidiate -->
+      <xacro:if value="${key == 2}">
+        <inertial>
+          <mass value="0.1"/>
+          <origin xyz="0 0 0" rpy="0 0 0"/>
+          <inertia ixx="55.59e-6" iyy="146.36e-6" izz="154.18e-6"
+                   ixy="-47.23e-6" ixz="1.16e-6" iyz="1.00e-6"/>
+        </inertial>
+      </xacro:if>
+      <!-- finger platform no finger (CURRENTLY COPY OF ABOVE) -->
+      <xacro:if value="${key == 3}">
+        <inertial>
+          <mass value="0.1"/>
+          <origin xyz="0 0 0" rpy="0 0 0"/>
+          <inertia ixx="55.59e-6" iyy="146.36e-6" izz="154.18e-6"
+                   ixy="-47.23e-6" ixz="1.16e-6" iyz="1.00e-6"/>
+        </inertial>
+      </xacro:if>
+      <!-- finger platform with finger -->
+      <xacro:if value="${key == 4}">
+        <inertial>
+          <mass value="0.2"/>
+          <origin xyz="0 0 0" rpy="0 0 0"/>
+          <inertia ixx="283.44e-6" iyy="1.38e-3" izz="1.60e-3"
+                   ixy="-567.23e-6" ixz="-6.59e-6" iyz="2.40e-6"/>
+        </inertial>
+      </xacro:if>
+      <!-- palm (CURRENTLY GUESSED)-->
+      <xacro:if value="${key == 5}">
+        <inertial>
+          <mass value="0.05"/>
+          <origin xyz="0 0 0" rpy="0 0 0"/>
+          <inertia ixx="10.0e-6" iyy="10.0e-6" izz="10.0e-6"
+                   ixy="0.0" ixz="0.0" iyz="0.0"/>
+        </inertial>
+      </xacro:if>
+    </xacro:macro>
+    <!-- END OF PARAMETER TO BE SET BY HAND -->
+    <!-- Constants for specifying finger start position, no need to change -->
+    <xacro:property name="radius" value="0.0"/>
+    <xacro:property name="angle" value="0.0"/>
+    <!-- Simplistic inertia macro for Gazebo -->
     <xacro:macro name="default_inertial" params="mass">
       <inertial>
@@ -33,52 +83,4 @@
                 ixy="0.00" iyz="0.00" ixz="0.00" />
       </inertial>
-    </xacro:macro>
-    <!-- inertias from solidworks -->
-    <xacro:macro name="set_inertia" params="key">
-      <!-- Base-->
-      <xacro:if value="${key == 1}">
-        <inertial>
-          <mass value="1.5"/>
-          <origin xyz="0 0 ${25*0.001}" rpy="${pi} 0 0"/>
-          <inertia ixx="9.95e-3" iyy="10.08e-3" izz="5.13e-3"
-                   ixy="2.73e-6" ixz="-14.32e-6" iyz="121.38e-6"/>
-        </inertial>
-      </xacro:if>
-      <!-- finger intermidiate -->
-      <xacro:if value="${key == 2}">
-        <inertial>
-          <mass value="0.1"/>
-          <origin xyz="0 0 0" rpy="0 0 0"/>
-          <inertia ixx="55.59e-6" iyy="146.36e-6" izz="154.18e-6"
-                   ixy="-47.23e-6" ixz="1.16e-6" iyz="1.00e-6"/>
-        </inertial>
-      </xacro:if>
-      <!-- finger platform no finger (CURRENTLY COPY OF ABOVE) -->
-      <xacro:if value="${key == 3}">
-        <inertial>
-          <mass value="0.1"/>
-          <origin xyz="0 0 0" rpy="0 0 0"/>
-          <inertia ixx="55.59e-6" iyy="146.36e-6" izz="154.18e-6"
-                   ixy="-47.23e-6" ixz="1.16e-6" iyz="1.00e-6"/>
-        </inertial>
-      </xacro:if>
-      <!-- finger platform with finger -->
-      <xacro:if value="${key == 4}">
-        <inertial>
-          <mass value="0.2"/>
-          <origin xyz="0 0 0" rpy="0 0 0"/>
-          <inertia ixx="283.44e-6" iyy="1.38e-3" izz="1.60e-3"
-                   ixy="-567.23e-6" ixz="-6.59e-6" iyz="2.40e-6"/>
-        </inertial>
-      </xacro:if>
-      <!-- palm (CURRENTLY GUESSED)-->
-      <xacro:if value="${key == 5}">
-        <inertial>
-          <mass value="0.05"/>
-          <origin xyz="0 0 0" rpy="0 0 0"/>
-          <inertia ixx="10.0e-6" iyy="10.0e-6" izz="10.0e-6"
-                   ixy="0.0" ixz="0.0" iyz="0.0"/>
-        </inertial>
-      </xacro:if>
     </xacro:macro>
     <!-- BASE LINK -->

File: gripper_v2/gripper_description/xacro/gripper.segmented_fingers.xacro (robot description, xacro)
@@ -2,4 +2,5 @@
 <robot xmlns:xacro="http://ros.org/wiki/xacro">
   <xacro:macro name="segmented_finger" params="prefix num_segments torsion">
+  	<!-- PARAMETERS TO BE SET BY HAND -->
     <!-- User defined variables -->
     <xacro:property name="finger_length_mm" value="190.0"/>
@@ -34,4 +35,5 @@
     <xacro:property name="joint_friction" value="0.0"/>
     <xacro:property name="joint_damping" value="0.001"/>
+    <!-- END OF PARAMETERS TO BE SET BY HAND -->
     <!-- Automatially calculated variables -->
     <xacro:property name="finger_length" value="${finger_length_mm * 0.001}"/>

File: gripper_v2/gripper_description/xacro/gripper.xacro (robot description, xacro)
@@ -2,7 +2,14 @@
 <robot name="gripper" xmlns:xacro="http://wiki.ros.org/xacro">
 	<xacro:macro name="add_gripper">
+		<!-- PARAMETERS TO BE SET BY HAND -->
+		<!-- xyz values to connect the segmented finger to the finger platform -->
+		<!-- TODO verfiy these values -->
+		<xacro:property name="x_fix" value="0.129"/>
+		<xacro:property name="y_fix" value="-0.007"/>
+		<xacro:property name="z_fix" value="0"/>
+		<!-- END OF PARAMETERS TO BE SET BY HAND -->
 		<!-- load information from the gripper yaml file -->
 		<xacro:property name="filename" value="$(find gripper_description)/config/gripper.yaml"/>
-		<xacro:property name="dictionary" value="${load_yaml(filename)}"/>
+		<xacro:property name="dictionary" value="${xacro.load_yaml(filename)}"/>
 		<xacro:property name="is_segmented" value="${dictionary['gripper_config']['is_segmented']}"/>
 		<xacro:property name="num_segments" value="${dictionary['gripper_config']['num_segments']}"/>
@@ -25,17 +32,16 @@
 		  <xacro:gazebo_plugin/>
 		  <!-- attach them to the gripper -->
-		  <!-- TODO verify these values -->
 		  <joint name="to_segmented_finger_1" type="fixed">
-		    <origin xyz="0.129 -0.007 0" rpy="${pi/2} 0 0"/>
+		    <origin xyz="${x_fix} ${y_fix} ${z_fix}" rpy="${pi/2} 0 0"/>
 		    <parent link="finger_1"/>
 		    <child link="finger_1_segment_link_1"/>
 		  </joint>
 		  <joint name="to_segmented_finger_2" type="fixed">
-		    <origin xyz="0.129 -0.007 0" rpy="${pi/2} 0 0"/>
+		    <origin xyz="${x_fix} ${y_fix} ${z_fix}" rpy="${pi/2} 0 0"/>
 		    <parent link="finger_2"/>
 		    <child link="finger_2_segment_link_1"/>
 		  </joint>
 		  <joint name="to_segmented_finger_3" type="fixed">
-		    <origin xyz="0.129 -0.007 0" rpy="${pi/2} 0 0"/>
+		    <origin xyz="${x_fix} ${y_fix} ${z_fix}" rpy="${pi/2} 0 0"/>
 		    <parent link="finger_3"/>
 		    <child link="finger_3_segment_link_1"/>

File: gripper_v2/gripper_description/xacro/panda.control.xacro (robot description, xacro)
@@ -1,3 +1,3 @@
-<?xml version="1.0"?>
+<?xml version='1.0' encoding='UTF-8'?>
 <robot xmlns:xacro="http://www.ros.org/wiki/xacro">
     <xacro:macro name="panda_control" params="arm_id">

File: gripper_v2/gripper_description/xacro/panda.main.xacro (robot description, xacro)
@@ -11,7 +11,12 @@
       </joint>
     </xacro:unless> -->
-    <!-- added a 5.0N friction tag in the joint macro below -->
+    <!-- PARAMETERS TO SET BY HAND -->
+    <!-- adjustable properties -->
     <xacro:property name="joint_damping" value="1.0"/>
-    <xacro:property name="joint_friction" value="0.0"/>
+    <xacro:property name="joint_friction" value="0.1"/>
+    <xacro:property name="large_limit_effort" value="87"/>
+    <xacro:property name="small_limit_effort" value="12"/>
+    <xacro:property name="realistic_inertia" value="true"/>
+    <!-- END OF PARAMETERS TO SET BY HAND -->
     <!-- written by luke based off: https://github.com/justagist/franka_panda_description/blob/master/robots/panda_arm.xacro -->
     <xacro:macro name="retrieve_inertia" params="link_number">
@@ -63,6 +68,10 @@
           <origin xyz="0 0 0" rpy="0 0 0" />
           <mass value="${mass}"/>
-          <xacro:retrieve_inertia link_number="${number}"/>
-          <!-- <inertia ixx="3e-1" ixy="0.0" ixz="0.0" iyy="3e-1" iyz="0.0" izz="3e-1" /> -->
+          <xacro:if value="${realistic_inertia}">
+          	<xacro:retrieve_inertia link_number="${number}"/>
+          </xacro:if>
+          <xacro:unless value="${realistic_inertia}">
+          	<inertia ixx="3e-1" ixy="0.0" ixz="0.0" iyy="3e-1" iyz="0.0" izz="3e-1" />
+          </xacro:unless>
         </inertial>
       </link>
@@ -88,42 +97,61 @@
       </joint>
     </xacro:macro>
-    <xacro:arm_link number="0" visual_mesh="package://${mesh_folder}/visual/link0.dae"
-      collision_mesh="package://${mesh_folder}/collision/link0.stl" mass="3.06"/>
-    <xacro:arm_link number="1" visual_mesh="package://${mesh_folder}/visual/link1.dae"
-      collision_mesh="package://${mesh_folder}/collision/link1.stl" mass="2.34"/>
-    <xacro:arm_link number="2" visual_mesh="package://${mesh_folder}/visual/link2.dae"
-      collision_mesh="package://${mesh_folder}/collision/link2.stl" mass="2.36"/>
-    <xacro:arm_link number="3" visual_mesh="package://${mesh_folder}/visual/link3.dae"
-      collision_mesh="package://${mesh_folder}/collision/link3.stl" mass="2.38"/>
-    <xacro:arm_link number="4" visual_mesh="package://${mesh_folder}/visual/link4.dae"
-      collision_mesh="package://${mesh_folder}/collision/link4.stl" mass="2.43"/>
-    <xacro:arm_link number="5" visual_mesh="package://${mesh_folder}/visual/link5.dae"
-      collision_mesh="package://${mesh_folder}/collision/link5.stl" mass="3.5"/>
-    <xacro:arm_link number="6" visual_mesh="package://${mesh_folder}/visual/link6.dae"
-      collision_mesh="package://${mesh_folder}/collision/link6.stl" mass="1.47"/>
-    <xacro:arm_link number="7" visual_mesh="package://${mesh_folder}/visual/link7.dae"
-      collision_mesh="package://${mesh_folder}/collision/link7.stl" mass="0.45"/>
+    <!-- original working mesh links -->
+<!--    <xacro:arm_link number="0" visual_mesh="package://${mesh_folder}/visual/link0.dae"-->
+<!--      collision_mesh="package://${mesh_folder}/collision/link0.stl" mass="3.06"/>-->
+<!--    <xacro:arm_link number="1" visual_mesh="package://${mesh_folder}/visual/link1.dae"-->
+<!--      collision_mesh="package://${mesh_folder}/collision/link1.stl" mass="2.34"/>-->
+<!--    <xacro:arm_link number="2" visual_mesh="package://${mesh_folder}/visual/link2.dae"-->
+<!--      collision_mesh="package://${mesh_folder}/collision/link2.stl" mass="2.36"/>-->
+<!--    <xacro:arm_link number="3" visual_mesh="package://${mesh_folder}/visual/link3.dae"-->
+<!--      collision_mesh="package://${mesh_folder}/collision/link3.stl" mass="2.38"/>-->
+<!--    <xacro:arm_link number="4" visual_mesh="package://${mesh_folder}/visual/link4.dae"-->
+<!--      collision_mesh="package://${mesh_folder}/collision/link4.stl" mass="2.43"/>-->
+<!--    <xacro:arm_link number="5" visual_mesh="package://${mesh_folder}/visual/link5.dae"-->
+<!--      collision_mesh="package://${mesh_folder}/collision/link5.stl" mass="3.5"/>-->
+<!--    <xacro:arm_link number="6" visual_mesh="package://${mesh_folder}/visual/link6.dae"-->
+<!--      collision_mesh="package://${mesh_folder}/collision/link6.stl" mass="1.47"/>-->
+<!--    <xacro:arm_link number="7" visual_mesh="package://${mesh_folder}/visual/link7.dae"-->
+<!--      collision_mesh="package://${mesh_folder}/collision/link7.stl" mass="0.45"/>-->
+<!--     <xacro:arm_link number="8"/>-->
+		<!-- testing new mesh files all being stl and all being in top level of folder for mujoco -->
+		<xacro:arm_link number="0" visual_mesh="package://${mesh_folder}/panda visual link0.stl"
+      collision_mesh="package://${mesh_folder}/panda collision link0.stl" mass="3.06"/>
+    <xacro:arm_link number="1" visual_mesh="package://${mesh_folder}/panda visual link1.stl"
+      collision_mesh="package://${mesh_folder}/panda collision link1.stl" mass="2.34"/>
+    <xacro:arm_link number="2" visual_mesh="package://${mesh_folder}/panda visual link2.stl"
+      collision_mesh="package://${mesh_folder}/panda collision link2.stl" mass="2.36"/>
+    <xacro:arm_link number="3" visual_mesh="package://${mesh_folder}/panda visual link3.stl"
+      collision_mesh="package://${mesh_folder}/panda collision link3.stl" mass="2.38"/>
+    <xacro:arm_link number="4" visual_mesh="package://${mesh_folder}/panda visual link4.stl"
+      collision_mesh="package://${mesh_folder}/panda collision link4.stl" mass="2.43"/>
+    <xacro:arm_link number="5" visual_mesh="package://${mesh_folder}/panda visual link5.stl"
+      collision_mesh="package://${mesh_folder}/panda collision link5.stl" mass="3.5"/>
+    <xacro:arm_link number="6" visual_mesh="package://${mesh_folder}/panda visual link6.stl"
+      collision_mesh="package://${mesh_folder}/panda collision link6.stl" mass="1.47"/>
+    <xacro:arm_link number="7" visual_mesh="package://${mesh_folder}/panda visual link7.stl"
+      collision_mesh="package://${mesh_folder}/panda collision link7.stl" mass="0.45"/>
      <xacro:arm_link number="8"/>
      <!-- joint6 limit lower = -0.0175 -->
     <xacro:arm_joint name="${arm_id}_joint1" type="revolute" soft_lower_limit="-2.8973" soft_upper_limit="2.8973"
-      rpy="0 0 0" xyz="0 0 0.333" parent_link="${arm_id}_link0" child_link="${arm_id}_link1" limit_effort="87"
+      rpy="0 0 0" xyz="0 0 0.333" parent_link="${arm_id}_link0" child_link="${arm_id}_link1" limit_effort="${large_limit_effort}"
       limit_lower="-2.8973" limit_upper="2.8973" limit_velocity="2.1750"/>
     <xacro:arm_joint name="${arm_id}_joint2" type="revolute" soft_lower_limit="-1.7628" soft_upper_limit="1.7628"
-      rpy="${-pi/2} 0 0" xyz="0 0 0" parent_link="${arm_id}_link1" child_link="${arm_id}_link2" limit_effort="87"
+      rpy="${-pi/2} 0 0" xyz="0 0 0" parent_link="${arm_id}_link1" child_link="${arm_id}_link2" limit_effort="${large_limit_effort}"
       limit_lower="-1.7628" limit_upper="1.7628" limit_velocity="2.1750"/>
     <xacro:arm_joint name="${arm_id}_joint3" type="revolute" soft_lower_limit="-2.8973" soft_upper_limit="2.8973"
-      rpy="${pi/2} 0 0" xyz="0 -0.316 0" parent_link="${arm_id}_link2" child_link="${arm_id}_link3" limit_effort="87"
+      rpy="${pi/2} 0 0" xyz="0 -0.316 0" parent_link="${arm_id}_link2" child_link="${arm_id}_link3" limit_effort="${large_limit_effort}"
       limit_lower="-2.8973" limit_upper="2.8973" limit_velocity="2.1750"/>
     <xacro:arm_joint name="${arm_id}_joint4" type="revolute" soft_lower_limit="-3.0718" soft_upper_limit="-0.0698"
-      rpy="${pi/2} 0 0" xyz="0.0825 0 0" parent_link="${arm_id}_link3" child_link="${arm_id}_link4" limit_effort="87"
+      rpy="${pi/2} 0 0" xyz="0.0825 0 0" parent_link="${arm_id}_link3" child_link="${arm_id}_link4" limit_effort="${large_limit_effort}"
       limit_lower="-3.0718" limit_upper="-0.0698" limit_velocity="2.1750"/>
     <xacro:arm_joint name="${arm_id}_joint5" type="revolute" soft_lower_limit="-2.8973" soft_upper_limit="2.8973"
-      rpy="${-pi/2} 0 0" xyz="-0.0825 0.384 0" parent_link="${arm_id}_link4" child_link="${arm_id}_link5" limit_effort="12"
+      rpy="${-pi/2} 0 0" xyz="-0.0825 0.384 0" parent_link="${arm_id}_link4" child_link="${arm_id}_link5" limit_effort="${small_limit_effort}"
       limit_lower="-2.8973" limit_upper="2.8973" limit_velocity="2.6100"/>
     <xacro:arm_joint name="${arm_id}_joint6" type="revolute" soft_lower_limit="-0.0175" soft_upper_limit="3.7525"
-      rpy="${pi/2} 0 0" xyz="0 0 0" parent_link="${arm_id}_link5" child_link="${arm_id}_link6" limit_effort="12"
+      rpy="${pi/2} 0 0" xyz="0 0 0" parent_link="${arm_id}_link5" child_link="${arm_id}_link6" limit_effort="${small_limit_effort}"
       limit_lower="-0.0175" limit_upper="3.7525" limit_velocity="2.6100"/>
     <xacro:arm_joint name="${arm_id}_joint7" type="revolute" soft_lower_limit="-2.8973" soft_upper_limit="2.8973"
-      rpy="${pi/2} 0 0" xyz="0.088 0 0" parent_link="${arm_id}_link6" child_link="${arm_id}_link7" limit_effort="12"
+      rpy="${pi/2} 0 0" xyz="0.088 0 0" parent_link="${arm_id}_link6" child_link="${arm_id}_link7" limit_effort="${small_limit_effort}"
       limit_lower="-2.8973" limit_upper="2.8973" limit_velocity="2.6100"/>
     <xacro:arm_joint name="${arm_id}_joint8" type="fixed" parent_link="${arm_id}_link7" child_link="${arm_id}_link8"
