Commit message: more

File: gripper_v2/gripper_description/xacro/semantic/add_gripper_config.xacro (robot description, xacro)
@@ -8,5 +8,5 @@
 		  <!-- retrieve info about the gripper -->
 		  <xacro:property name="filename" value="$(find gripper_description)/config/gripper.yaml"/>
-		  <xacro:property name="dictionary" value="${load_yaml(filename)}"/>
+		  <xacro:property name="dictionary" value="${xacro.load_yaml(filename)}"/>
 		  <xacro:property name="is_segmented" value="${dictionary['gripper_config']['is_segmented']}"/>
 		  <xacro:property name="num_segments" value="${dictionary['gripper_config']['num_segments']}"/>

File: gripper_v2/gripper_description/xacro/semantic/add_panda_config.xacro (robot description, xacro)
@@ -15,6 +15,6 @@
 		      <joint name="panda_joint6" />
 		      <joint name="panda_joint7" />
-		      <joint name="panda_joint8" />
-		      <joint name="world_to_base" />
+		      <joint name="world_to_base"/>
+		      <link name="panda_link8"/>
 		  </group>
 		  <!-- define a pose for this group -->

File: gripper_v2/gripper_description/xacro/semantic/panda_and_gripper.semantic.xacro (robot description, xacro)
@@ -9,6 +9,6 @@
 		<xacro:include filename="$(find gripper_description)/xacro/semantic/add_panda_config.xacro"/>
 		<!-- run the macros -->
+		<xacro:add_panda_config/>
 		<xacro:add_gripper_config/>
-		<xacro:add_panda_config/>
     <!--GROUPS: Representation of a set of joints and links. This can be useful for specifying DOF to plan for, defining arms, end effectors, etc-->
     <!--LINKS: When a link is specified, the parent joint of that link (if it exists) is automatically included-->
@@ -21,5 +21,5 @@
     </group>
     <!--END EFFECTOR: Purpose: Represent information about an end effector.-->
-    <end_effector name="gripper" parent_link="panda_link8" group="gripper" />
+    <end_effector name="mygripper" parent_link="panda_link8" group="gripper" parent_group="panda_arm" />
     <!--DISABLE COLLISIONS: By default it is assumed that any link of the robot could potentially come into collision with any other link in the robot. This tag disables collision checking between a specified pair of links. -->
     <disable_collisions link1="finger_1_intermediate" link2="panda_link3" reason="Never" />
