Commit message: model updates

File: gripper_v2/gripper_description/urdf/mujoco/gripper_task.urdf (robot description, URDF)
Before this commit: robot gripper, 42 links, 41 joints
Joints:
- joint world_to_base: origin xyz=0 0 1 rpy=3.14159265359 0 0 -> xyz=0 0 0.325 rpy=3.14159265359 0 0

File: gripper_v2/gripper_description/urdf/mujoco/panda_and_gripper_mujoco.urdf (robot description, URDF)
Before this commit: robot panda_and_gripper, 51 links, 50 joints
Links:
- link gripper_base_link: geometry collision cylinder length=0.1 radius=0.03; visual mesh filename=package://gripper_description/meshes/main body visual.STL

File: gripper_v2/gripper_description/urdf/mujoco/xacro/mujoco.xacro (robot description, xacro)
@@ -2,25 +2,12 @@
 <robot name="gripper" xmlns:xacro="http://wiki.ros.org/xacro">
 	<xacro:macro name="mujoco_settings">
-<!--		<mujoco>-->
-			<!-- compiler settings: required -->
-<!--			<compiler-->
-<!--				meshdir="./meshes_mujoco/"-->
-<!--				balanceinertia="true"-->
-<!--				discardvisual="false"-->
-<!--			/>-->
-			<!-- defaults 500, 100 need to be adjusted -->
-<!--			<size njmax="1400" nconmax="500"/>-->
-			<!-- set inital pose keyframe DOESN'T WORK WITH URDF PARSER -->
-			<!-- <keyframe>
-				<key name="initial pose"
-						time="0"
-						qpos="0 0 0 0 0 0.6 0
-									140e-3 0    0 0 0 0 0 0 0 0 0
-									140e-3 0    0 0 0 0 0 0 0 0 0
-									140e-3 0    0 0 0 0 0 0 0 0 0
-									0"
-				/>
-			</keyframe> -->
-<!--		</mujoco>-->
+		<mujoco>
+			<compiler
+				meshdir="./meshes_mujoco/"
+				balanceinertia="true"
+				discardvisual="false"
+			/>
+			<size njmax="1400" nconmax="500"/>
+		</mujoco>
 	</xacro:macro>
 </robot>

File: gripper_v2/gripper_description/xacro/gripper.main.xacro (robot description, xacro)
@@ -95,5 +95,6 @@
       <collision>
         <geometry>
-          <mesh filename="package://gripper_description/meshes/main body collision.STL"/>
+<!--          <mesh filename="package://gripper_description/meshes/main body collision.STL"/>-->
+					<cylinder length="0.1" radius="0.03"/>
         </geometry>
       </collision>

File: gripper_v2/gripper_description/xacro/gripper.segmented_fingers.xacro (robot description, xacro)
@@ -34,5 +34,5 @@
     <!-- these are implemented in the <dynamics> tags in each joint -->
     <xacro:property name="joint_friction" value="0.0"/>
-    <xacro:property name="joint_damping" value="0.001"/>
+    <xacro:property name="joint_damping" value="0.01"/>
     <!-- END OF PARAMETERS TO BE SET BY HAND -->
     <!-- Automatially calculated variables -->

Commit message: updates

File: gripper_v2/gripper_description/urdf/mujoco/gripper_task.urdf (robot description, URDF)
Before this commit: robot gripper_task, 42 links, 41 joints
Joints:
- joint world_to_base: axis (none) -> 0 0 1; limit (none) -> lower=-1 upper=1 effort=1e3 velocity=1; origin xyz=0 0 0.325 rpy=3.14159265359 0 0 -> xyz=0 0 0.335 rpy=3.14159265359 0 0; type fixed -> prismatic

File: gripper_v2/gripper_description/urdf/mujoco/xacro/gripper_task.urdf.xacro (robot description, xacro)
@@ -9,8 +9,14 @@
   <!-- attach gripper to the ground for gazebo -->
 	<link name="world"/>
-	<joint name="world_to_base" type="fixed">
-		<origin xyz="0 0 0.325" rpy="${pi} 0 0"/>
+	<joint name="world_to_base" type="prismatic">
+		<origin xyz="0 0 0.335" rpy="${pi} 0 0"/> <!-- 0.325 is fingertips just not touching-->
+		<axis xyz="0 0 1" rpy="0 0 0"/>
 		<parent link="world"/>
 		<child link="gripper_base_link"/>
+		<limit effort="1e3"
+        			 lower="-1"
+        			 upper="1"
+        			 velocity="1"/>
+    <dynamics damping="1"/>
 	</joint>
 </robot>

File: gripper_v2/gripper_description/xacro/gripper.segmented_fingers.xacro (robot description, xacro)
@@ -43,6 +43,4 @@
     <xacro:property name="hook_length" value="${hook_length_mm * 0.001}"/>
     <xacro:property name="hook_angle" value="${(hook_angle_d / 180.0) * 3.1415926535897}"/>
-    <!-- <xacro:property name="joint_friction" value="${total_friction / num_segments}"/>
-    <xacro:property name="joint_damping" value="${total_damping * num_segments}"/> -->
     <!-- find inertia of each segment -->
     <xacro:property name="finger_mass" value="${finger_mass_g * 0.001}"/>
