Commit message: 795 object set

File: gripper_v2/gripper_description/urdf/mujoco/mjcf_files/mjcf_include/create_objects.xacro (robot description, xacro)
@@ -1,5 +1,5 @@
 <mujoco xmlns:xacro="http://ros.org/wiki/xacro">
   <!-- 1. Extract dionary of settings -->
-  <xacro:property name="yamlpath" value="/home/luke/gripper_repo_ws/src/gripper_v2/gripper_description/urdf/mujoco/mjcf_include"/>
+  <xacro:property name="yamlpath" value="/home/luke/gripper_repo_ws/src/gripper_v2/gripper_description/urdf/mujoco/mjcf_files/mjcf_include"/>
   <xacro:property name="yamlname" value="define_objects.yaml"/>
   <xacro:property name="mydict" value="${xacro.load_yaml(yamlpath + '/' + yamlname)}"/>
